File: _saved_mars-aqua-adapter.sch (KiCad schematic (older format))
At the start: 40 parts, among them J1 Conn_01x03, J2 Conn_01x03, J3 Conn_01x04, J4 Conn_01x04, J5 Conn_01x03, J6 Conn_01x03, Q2 Q_PNP_BEC, U1 LM358, U2 LM393

Commit message: board layout
Parts:
- gave numbers to parts that had none: 1
Changed lines of the file:
@@
 $EndComp
 $Comp
-L Device:Q_PNP_BEC Q?
+L Device:Q_PNP_BEC Q1
 U 1 1 5C86EAA4
 P 8200 2600
-F 0 "Q?" H 8391 2554 50  0000 L CNN
+F 0 "Q1" H 8391 2554 50  0000 L CNN
 F 1 "Q_PNP_BEC" H 8391 2645 50  0000 L CNN
 F 2 "Package_TO_SOT_SMD:SOT-23" H 8400 2700 50  0001 C CNN
