File: mars-aqua-adapter.sch (KiCad schematic (older format))
At the start: 49 parts, among them J1 Conn_01x03, J2 Conn_01x03, J3 Conn_01x04, J4 Conn_01x04, J5 Conn_01x03, J6 Conn_01x03, Q1 Q_PNP_BEC, Q2 Q_PNP_BEC, Q3 Q_NPN_BEC, Q4 Q_NPN_BEC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

Commit message: gerber updates
Parts:
- removed D1: TL431DBZ, Package_TO_SOT_SMD:SOT-23, symbol Reference_Voltage:TL431DBZ
- added D1: TL432DBZ, Package_TO_SOT_SMD:SOT-23, symbol Reference_Voltage:TL432DBZ
Connections:
- net GND: now also D1.3 (A)
- net Vref: now also D1.2 (K)
- net at R27.1, R28.2: now also D1.1 (REF)
Changed lines of the file:
@@
 	7350 4400 7350 4900
-$Comp
-L Reference_Voltage:TL431DBZ D1
-U 1 1 5D055AD5
-P 5050 1350
-F 0 "D1" V 5096 1280 50  0000 R CNN
-F 1 "TL431DBZ" V 5005 1280 50  0000 R CNN
-F 2 "Package_TO_SOT_SMD:SOT-23" H 5050 1200 50  0001 C CIN
-F 3 "http://www.ti.com/lit/ds/symlink/tl431.pdf" H 5050 1350 50  0001 C CIN
-	1    5050 1350
-	0    -1   -1   0
-$EndComp
 $Comp
 L Device:R_US R27
@@
 Wire Wire Line
 	5600 1650 5050 1650
+$Comp
+L Reference_Voltage:TL432DBZ D1
+U 1 1 5D1EF6F2
+P 5050 1350
+F 0 "D1" V 5096 1280 50  0000 R CNN
+F 1 "TL432DBZ" V 5005 1280 50  0000 R CNN
+F 2 "Package_TO_SOT_SMD:SOT-23" H 5050 1200 50  0001 C CIN
+F 3 "http://www.ti.com/lit/ds/symlink/tl431.pdf" H 5050 1350 50  0001 C CIN
+	1    5050 1350
+	0    -1   -1   0
+$EndComp
 $EndSCHEMATC

Commit message: update feedback and regulator values
Parts:
- R20, R7: value 1M -> 5.1M
- R29: value 22 -> 470
Changed lines of the file:
@@
 P 5050 900
 F 0 "R29" H 5118 946 50  0000 L CNN
-F 1 "22" H 5118 855 50  0000 L CNN
+F 1 "470" H 5118 855 50  0000 L CNN
 F 2 "Resistor_SMD:R_0603_1608Metric_Pad1.05x0.95mm_HandSolder" V 5090 890 50  0001 C CNN
 F 3 "~" H 5050 900 50  0001 C CNN
@@
 P 7050 4400
 F 0 "R7" V 6845 4400 50  0000 C CNN
-F 1 "1M" V 6936 4400 50  0000 C CNN
+F 1 "5.1M" V 6936 4400 50  0000 C CNN
 F 2 "Resistor_SMD:R_0603_1608Metric_Pad1.05x0.95mm_HandSolder" V 7090 4390 50  0001 C CNN
 F 3 "~" H 7050 4400 50  0001 C CNN
@@
 P 7100 2100
 F 0 "R20" V 6895 2100 50  0000 C CNN
-F 1 "1M" V 6986 2100 50  0000 C CNN
+F 1 "5.1M" V 6986 2100 50  0000 C CNN
 F 2 "Resistor_SMD:R_0603_1608Metric_Pad1.05x0.95mm_HandSolder" V 7140 2090 50  0001 C CNN
 F 3 "~" H 7100 2100 50  0001 C CNN

Commit message: Update values
Parts:
- R19, R6: value 100k -> 10k
- R20, R7: value 5.1M -> 1M
Changed lines of the file:
@@
 P 7050 4400
 F 0 "R7" V 6845 4400 50  0000 C CNN
-F 1 "5.1M" V 6936 4400 50  0000 C CNN
+F 1 "1M" V 6936 4400 50  0000 C CNN
 F 2 "Resistor_SMD:R_0603_1608Metric_Pad1.05x0.95mm_HandSolder" V 7090 4390 50  0001 C CNN
 F 3 "~" H 7050 4400 50  0001 C CNN
@@
 P 7100 2100
 F 0 "R20" V 6895 2100 50  0000 C CNN
-F 1 "5.1M" V 6986 2100 50  0000 C CNN
+F 1 "1M" V 6986 2100 50  0000 C CNN
 F 2 "Resistor_SMD:R_0603_1608Metric_Pad1.05x0.95mm_HandSolder" V 7140 2090 50  0001 C CNN
 F 3 "~" H 7100 2100 50  0001 C CNN
@@
 P 6400 4400
 F 0 "R6" V 6195 4400 50  0000 C CNN
-F 1 "100k" V 6286 4400 50  0000 C CNN
+F 1 "10k" V 6286 4400 50  0000 C CNN
 F 2 "Resistor_SMD:R_0603_1608Metric_Pad1.05x0.95mm_HandSolder" V 6440 4390 50  0001 C CNN
 F 3 "~" H 6400 4400 50  0001 C CNN
@@
 P 6400 2100
 F 0 "R19" V 6195 2100 50  0000 C CNN
-F 1 "100k" V 6286 2100 50  0000 C CNN
+F 1 "10k" V 6286 2100 50  0000 C CNN
 F 2 "Resistor_SMD:R_0603_1608Metric_Pad1.05x0.95mm_HandSolder" V 6440 2090 50  0001 C CNN
 F 3 "~" H 6400 2100 50  0001 C CNN
